File: f030dev1.kicad_pcb (KiCad board)
At the start: 2 copper layers, 5 parts, among them J1 Conn_01x10_Pin, J2 Conn_01x03_Pin, U1 STM32F030F4Px, U2 74HC595, U3 AMS1117-3.3

Commit message: в процесе
Parts:
- added J3: Conn_01x08_Pin, main:PinHeader_2x04_P2.54mm_Vertical, F.Cu at (152.5, 97.4)
- J1: footprint main:PinHeader_2x05_P2.00mm_Vertical -> main:PinHeader_2x05_P2.54mm_Vertical
- moved J1 1.49 mm to (172.5, 65.0)

Commit message: Старт
схему нужно проверять
Parts:
- removed the J1 at (172.5, 65.0)
- added C1: C_Polarized, Capacitor_THT:CP_Radial_D7.5mm_P2.50mm, F.Cu at (107.3, 76.8)
- added C2: C_Small, Capacitor_SMD:C_0805_2012Metric_Pad1.18x1.45mm_HandSolder, B.Cu at (139.7, 76.8)
- added C3: C_Small, Capacitor_SMD:C_0805_2012Metric_Pad1.18x1.45mm_HandSolder, B.Cu at (154.0, 65.0)
- added C4: C_Polarized, Capacitor_THT:CP_Radial_D7.5mm_P2.50mm, F.Cu at (120.7, 76.2)
- added J2: Conn_01x02_Pin, main:PinHeader_1x02_P2.54mm_Vertical, F.Cu at (108.6, 63.5)
- added J4: Conn_01x10_Pin, main:PinHeader_2x05_P2.54mm_Vertical, F.Cu at (167.5, 75.0)
- J3: value Conn_01x08_Pin -> Conn_01x06_Pin; footprint main:PinHeader_2x04_P2.54mm_Vertical -> main:PinHeader_1x06_P2.54mm_Vertical
- moved J1 37.6 mm to (137.7, 64.1), turned to 90 degrees
- moved J3 29.1 mm to (130.2, 78.7), turned to 180 degrees
- moved U2 22.9 mm to (120.0, 66.0)
- moved U3 14.0 mm to (157.5, 80.0), turned to 180 degrees
- moved U1 9.41 mm to (139.7, 70.5)
- renumbered J2 to J1, U3 to U2, U2 to U3
Connections:
- J1 pad 1: unconnected-(J2-Pin_1-Pad1) -> +3.3V
- J1 pad 2: unconnected-(J2-Pin_2-Pad2) -> RX
- J1 pad 3: unconnected-(J2-Pin_3-Pad3) -> GNDREF
- J3 pad 1: unconnected-(J3-Pin_1-Pad1) -> +3.3V
- J3 pad 2: unconnected-(J3-Pin_2-Pad2) -> button_1
- J3 pad 3: unconnected-(J3-Pin_3-Pad3) -> button_2
- J3 pad 4: unconnected-(J3-Pin_4-Pad4) -> button_3
- J3 pad 5: unconnected-(J3-Pin_5-Pad5) -> button_4
- J3 pad 6: unconnected-(J3-Pin_6-Pad6) -> GNDREF
- U1 pad 1: unconnected-(U1-BOOT0-Pad1) -> GNDREF
- U1 pad 10: unconnected-(U1-PA4-Pad10) -> button_4
- U1 pad 11: unconnected-(U1-PA5-Pad11) -> CS_595
- U1 pad 12: unconnected-(U1-PA6-Pad12) -> CLK_595
- U1 pad 13: unconnected-(U1-PA7-Pad13) -> DAT_595
- U1 pad 15: unconnected-(U1-VSS-Pad15) -> GNDREF
- U1 pad 16: unconnected-(U1-VDD-Pad16) -> +3.3V
- U1 pad 5: unconnected-(U1-VDDA-Pad5) -> +3.3V
- U1 pad 6: unconnected-(U1-PA0-Pad6) -> RX
- U1 pad 7: unconnected-(U1-PA1-Pad7) -> button_1
- U1 pad 8: unconnected-(U1-PA2-Pad8) -> button_2
- U1 pad 9: unconnected-(U1-PA3-Pad9) -> button_3
- U2 pad 1: unconnected-(U3-GND-Pad1) -> GNDREF
- U2 pad 2: unconnected-(U3-VO-Pad2) -> +3.3V
- U2 pad 3: unconnected-(U3-VI-Pad3) -> +5V
- U3 pad 1: unconnected-(U2-QB-Pad1) -> Net-(J4-Pin_2)
- U3 pad 10: unconnected-(U2-~{SRCLR}-Pad10) -> +3.3V
- U3 pad 11: unconnected-(U2-SRCLK-Pad11) -> CLK_595
- U3 pad 12: unconnected-(U2-RCLK-Pad12) -> CS_595
- U3 pad 13: unconnected-(U2-~{OE}-Pad13) -> GNDREF
- U3 pad 14: unconnected-(U2-SER-Pad14) -> DAT_595
- U3 pad 15: unconnected-(U2-QA-Pad15) -> Net-(J4-Pin_1)
- U3 pad 16: unconnected-(U2-VCC-Pad16) -> +3.3V
- U3 pad 2: unconnected-(U2-QC-Pad2) -> Net-(J4-Pin_3)
- U3 pad 3: unconnected-(U2-QD-Pad3) -> Net-(J4-Pin_4)
- U3 pad 4: unconnected-(U2-QE-Pad4) -> Net-(J4-Pin_5)
- U3 pad 5: unconnected-(U2-QF-Pad5) -> Net-(J4-Pin_6)
- U3 pad 6: unconnected-(U2-QG-Pad6) -> Net-(J4-Pin_7)
- U3 pad 7: unconnected-(U2-QH-Pad7) -> Net-(J4-Pin_8)
- U3 pad 8: unconnected-(U2-GND-Pad8) -> GNDREF
Other:
- board outline added: 72.4 x 33.3 mm
